Commit message: （feat）碰撞添加，地图添加，3d点云功能添加

File: 路径规划与SLAM/mid360_ws/src/bot_description/urdf/robot.urdf.xacro (robot description, xacro)
@@ -4,7 +4,9 @@
   <xacro:arg name="camera_info_topic" default="/camera/camera_info"/>
   <xacro:arg name="mid360_topic" default="/mid360_points"/>
+  <xacro:arg name="laser_topic" default="/laser_points"/>
   <xacro:include filename="$(find bot_description)/urdf/base.urdf.xacro"/>
   <xacro:include filename="$(find bot_description)/urdf/camera.xacro"/>
   <xacro:include filename="$(find bot_description)/urdf/mid360_mount.xacro"/>
+  <xacro:include filename="$(find bot_description)/urdf/laser.xacro"/>
   <xacro:base/>
   <xacro:camera
@@ -14,5 +16,6 @@
     info_topic="$(arg camera_info_topic)"
     update_rate="10.0">
-    <origin xyz="0.30 0 0.32" rpy="0 0 0"/>
+    <!-- P把相机光学中心放在底盘前方、车顶上方。 -->
+    <origin xyz="0.46 0 0.35" rpy="0 0 0"/>
   </xacro:camera>
   <xacro:mid360
@@ -21,6 +24,15 @@
     topic="$(arg mid360_topic)"
     update_rate="10.0">
-    <origin xyz="0 0 0.30" rpy="0 0 0"/>
+    <!-- 高安装可以让 360 度扫描避开底盘顶部，避免遮挡。 -->
+    <origin xyz="0 0 0.52" rpy="0 0 0"/>
   </xacro:mid360>
+  <xacro:laser
+    name="laser"
+    parent="base_link"
+    topic="$(arg laser_topic)"
+    update_rate="15.0">
+    <!-- Front/top mount; the point cloud is published independently of MID360. -->
+    <origin xyz="0.18 0 0.48" rpy="0 0 0"/>
+  </xacro:laser>
   <!-- A simple planar controller makes cmd_vel/odom available in Gazebo. -->
   <gazebo>
